File: kzpe/kzpe.kicad_sch (KiCad schematic)
At the start: 22 parts, among them J1 Conn_12VIN, J2 Conn_FAN, J3 Conn_NTC, Q1 IRLL014TRPBF-BE3, U1 LM555xM, U2 TL081, U3 LF50ABDT-TR

Commit message: 0912
Parts:
- U1: footprint Package_SO:SOIC-8_3.9x4.9mm_P1.27mm -> kzpe_fp:SOIC127P600X175-8N
- U2: footprint Library:TL081 -> kzpe_fp:SOIC127P600X175-8N
Changed lines of the file:
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@@
 			)
 		)
-		(property "Footprint" "Library:TL081"
+		(property "Footprint" "kzpe_fp:SOIC127P600X175-8N"
 			(at 87.63 83.82 0)
 			(effects
@@
 			)
 		)
-		(property "Footprint" "Package_SO:SOIC-8_3.9x4.9mm_P1.27mm"
+		(property "Footprint" "kzpe_fp:SOIC127P600X175-8N"
 			(at 143.51 95.25 0)
 			(effects
